File: PCB/CredIT-Card.kicad_pcb (KiCad board)
At the start: 2 copper layers, 90 x 50 mm, 12 parts, among them J2 TE_3-1734839-0, J3 TE_2295018-2, SW1 SW_EG1215AA, SW2 2425578-1, SW3 2425578-1, U2 QFN-56-1EP_7x7mm_P0.4mm_EP3.2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

Commit message: Renamed PCB project
Parts:
- BT1: footprint myCC:RJD2032C1ST1 -> CredIT-Card:RJD2032C1ST1
- J2: footprint myCC:TE_3-1734839-0 -> CredIT-Card:TE_3-1734839-0
- J3: footprint myCC:TE_2295018-2 -> CredIT-Card:TE_2295018-2
- SW1: footprint myCC:SW_EG1215AA -> CredIT-Card:SW_EG1215AA
- SW2, SW3: footprint myCC:TE_2425578-1 -> CredIT-Card:TE_2425578-1
Changed lines of the file:
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@@
 		)
 	)
-	(footprint "myCC:RJD2032C1ST1"
+	(footprint "CredIT-Card:RJD2032C1ST1"
 		(layer "F.Cu")
 		(at 82 106)
@@
 			)
 		)
-		(property "Footprint" "myCC:RJD2032C1ST1"
+		(property "Footprint" "CredIT-Card:RJD2032C1ST1"
 			(at 0 0 0)
 			(unlocked yes)
@@
 			(thermal_bridge_angle 45)
 		)
-		(model "${KIPRJMOD}/myCC.pretty/RJD2032C1ST1.stp"
+		(model "${KIPRJMOD}/CredIT-Card.pretty/RJD2032C1ST1.stp"
 			(offset
 				(xyz 0 0 -4)
@@
 		)
 	)
-	(footprint "myCC:SW_EG1215AA"
+	(footprint "CredIT-Card:SW_EG1215AA"
 		(layer "F.Cu")
 		(at 72 94 -90)
@@
 			)
 		)
-		(property "Footprint" "myCC:SW_EG1215AA"
+		(property "Footprint" "CredIT-Card:SW_EG1215AA"
 			(at 0 0 -90)
 			(unlocked yes)
@@
 			(solder_mask_margin 0.102)
 		)
-		(model "${KIPRJMOD}/myCC.pretty/EG1215AA.step"
+		(model "${KIPRJMOD}/CredIT-Card.pretty/EG1215AA.step"
 			(offset
 				(xyz 0 0 1.5)
@@
 		)
 	)
-	(footprint "myCC:TE_2425578-1"
+	(footprint "CredIT-Card:TE_2425578-1"
 		(layer "B.Cu")
 		(at 136 69 180)
@@
 			)
 		)
-		(property "Footprint" "myCC:TE_2425578-1"
+		(property "Footprint" "CredIT-Card:TE_2425578-1"
 			(at 0 -5.3 0)
 			(unlocked yes)
@@
 			(thermal_bridge_angle 45)
 		)
-		(model "${KIPRJMOD}/myCC.pretty/c-2425578-1-a-3d.stp"
+		(model "${KIPRJMOD}/CredIT-Card.pretty/c-2425578-1-a-3d.stp"
 			(offset
 				(xyz 0 0.5 0.5)
@@
 		)
 	)
-	(footprint "myCC:TE_3-1734839-0"
+	(footprint "CredIT-Card:TE_3-1734839-0"
 		(layer "B.Cu")
 		(at 133 85 90)
@@
 			)
 		)
-		(property "Footprint" "myCC:TE_3-1734839-0"
+		(property "Footprint" "CredIT-Card:TE_3-1734839-0"
 			(at 0 0 -90)
 			(unlocked yes)
@@
 			(solder_mask_margin 0.102)
 		)
-		(model "${KIPRJMOD}/myCC.pretty/3-1734839-0.step"
+		(model "${KIPRJMOD}/CredIT-Card.pretty/3-1734839-0.step"
 			(offset
 				(xyz 0 -2.2 0)
@@
 		)
 	)
-	(footprint "myCC:TE_2295018-2"
+	(footprint "CredIT-Card:TE_2295018-2"
 		(layer "B.Cu")
 		(at 157.5 104.5 -90)
@@
 			)
 		)
-		(property "Footprint" "myCC:TE_2295018-2"
+		(property "Footprint" "CredIT-Card:TE_2295018-2"
 			(at 0 0 90)
 			(unlocked yes)
@@
 			(remove_unused_layers no)
 		)
-		(model "${KIPRJMOD}/myCC.pretty/2295018-2.step"
+		(model "${KIPRJMOD}/CredIT-Card.pretty/2295018-2.step"
 			(offset
 				(xyz 0 1.4 0)
@@
 		)
 	)
-	(footprint "myCC:TE_2425578-1"
+	(footprint "CredIT-Card:TE_2425578-1"
 		(layer "B.Cu")
 		(at 120 69 180)
@@
 			)
 		)
-		(property "Footprint" "myCC:TE_2425578-1"
+		(property "Footprint" "CredIT-Card:TE_2425578-1"
 			(at 0 -5.3 0)
 			(unlocked yes)
@@
 			(thermal_bridge_angle 45)
 		)
-		(model "${KIPRJMOD}/myCC.pretty/c-2425578-1-a-3d.stp"
+		(model "${KIPRJMOD}/CredIT-Card.pretty/c-2425578-1-a-3d.stp"
 			(offset
 				(xyz 0 0.5 0.5)
