File: PCB/POWER.kicad_sch (KiCad schematic)
At the start: 23 parts, among them U4 MAX77734BENP+, U5 TPSM83100

Commit message: Renamed PCB project
Parts:
- BT1: footprint myCC:RJD2032C1ST1 -> CredIT-Card:RJD2032C1ST1
- U4: footprint myCC:BGA20N40P4X5_196X222X50N -> CredIT-Card:BGA20N40P4X5_196X222X50N; symbol myCC:MAX77734BENP_ -> CredIT-Card:MAX77734BENP_
- U5: symbol myCC:XTPSM83100SIUR -> CredIT-Card:XTPSM83100SIUR
Changed lines of the file:
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@@
 	)
 	(symbol
-		(lib_id "myCC:MAX77734BENP_")
+		(lib_id "CredIT-Card:MAX77734BENP_")
 		(at 137.16 123.19 0)
 		(unit 1)
@@
 			)
 		)
-		(property "Footprint" "myCC:BGA20N40P4X5_196X222X50N"
+		(property "Footprint" "CredIT-Card:BGA20N40P4X5_196X222X50N"
 			(at 137.16 123.19 0)
 			(effects
@@
 		)
 		(instances
-			(project "myCC"
+			(project "CredIT-Card"
 				(path "/cf02616b-7563-498d-8298-4a13535fe00b/26667293-4bc7-42dd-80bc-5789f6d81738"
 					(reference "U4")
@@
 		)
 		(instances
-			(project "myCC"
+			(project "CredIT-Card"
 				(path "/cf02616b-7563-498d-8298-4a13535fe00b/26667293-4bc7-42dd-80bc-5789f6d81738"
 					(reference "#PWR057")
@@
 		)
 		(instances
-			(project "myCC"
+			(project "CredIT-Card"
 				(path "/cf02616b-7563-498d-8298-4a13535fe00b/26667293-4bc7-42dd-80bc-5789f6d81738"
 					(reference "#PWR043")
@@
 		)
 		(instances
-			(project "myCC"
+			(project "CredIT-Card"
 				(path "/cf02616b-7563-498d-8298-4a13535fe00b/26667293-4bc7-42dd-80bc-5789f6d81738"
 					(reference "#PWR0163")
@@
 		)
 		(instances
-			(project "myCC"
+			(project "CredIT-Card"
 				(path "/cf02616b-7563-498d-8298-4a13535fe00b/26667293-4bc7-42dd-80bc-5789f6d81738"
 					(reference "#PWR0164")
@@
 		)
 		(instances
-			(project "myCC"
+			(project "CredIT-Card"
 				(path "/cf02616b-7563-498d-8298-4a13535fe00b/26667293-4bc7-42dd-80bc-5789f6d81738"
 					(reference "#PWR063")
@@
 		)
 		(instances
-			(project "myCC"
+			(project "CredIT-Card"
 				(path "/cf02616b-7563-498d-8298-4a13535fe00b/26667293-4bc7-42dd-80bc-5789f6d81738"
 					(reference "#PWR0165")
@@
 		)
 		(instances
-			(project "myCC"
+			(project "CredIT-Card"
 				(path "/cf02616b-7563-498d-8298-4a13535fe00b/26667293-4bc7-42dd-80bc-5789f6d81738"
 					(reference "#PWR045")
@@
 		)
 		(instances
-			(project "myCC"
+			(project "CredIT-Card"
 				(path "/cf02616b-7563-498d-8298-4a13535fe00b/26667293-4bc7-42dd-80bc-5789f6d81738"
 					(reference "#PWR044")
@@
 			)
 		)
-		(property "Footprint" "myCC:RJD2032C1ST1 "
+		(property "Footprint" "CredIT-Card:RJD2032C1ST1 "
 			(at 116.84 41.656 90)
 			(effects
@@
 		)
 		(instances
-			(project "myCC"
+			(project "CredIT-Card"
 				(path "/cf02616b-7563-498d-8298-4a13535fe00b/26667293-4bc7-42dd-80bc-5789f6d81738"
 					(reference "BT1")
@@
 		)
 		(instances
-			(project "myCC"
+			(project "CredIT-Card"
 				(path "/cf02616b-7563-498d-8298-4a13535fe00b/26667293-4bc7-42dd-80bc-5789f6d81738"
 					(reference "#PWR052")
@@
 		)
 		(instances
-			(project "myCC"
+			(project "CredIT-Card"
 				(path "/cf02616b-7563-498d-8298-4a13535fe00b/26667293-4bc7-42dd-80bc-5789f6d81738"
 					(reference "C20")
@@
 		)
 		(instances
-			(project "myCC"
+			(project "CredIT-Card"
 				(path "/cf02616b-7563-498d-8298-4a13535fe00b/26667293-4bc7-42dd-80bc-5789f6d81738"
 					(reference "#PWR046")
@@
 		)
 		(instances
-			(project "myCC"
+			(project "CredIT-Card"
 				(path "/cf02616b-7563-498d-8298-4a13535fe00b/26667293-4bc7-42dd-80bc-5789f6d81738"
 					(reference "#PWR060")
@@
 		)
 		(instances
-			(project "myCC"
+			(project "CredIT-Card"
 				(path "/cf02616b-7563-498d-8298-4a13535fe00b/26667293-4bc7-42dd-80bc-5789f6d81738"
 					(reference "#PWR065")
@@
 		)
 		(instances
-			(project "myCC"
+			(project "CredIT-Card"
 				(path "/cf02616b-7563-498d-8298-4a13535fe00b/26667293-4bc7-42dd-80bc-5789f6d81738"
 					(reference "#PWR061")
@@
 		)
 		(instances
-			(project "myCC"
+			(project "CredIT-Card"
 				(path "/cf02616b-7563-498d-8298-4a13535fe00b/26667293-4bc7-42dd-80bc-5789f6d81738"
 					(reference "#PWR049")
@@
 		)
 		(instances
-			(project "myCC"
+			(project "CredIT-Card"
 				(path "/cf02616b-7563-498d-8298-4a13535fe00b/26667293-4bc7-42dd-80bc-5789f6d81738"
 					(reference "R12")
@@
 		)
 		(instances
-			(project "myCC"
+			(project "CredIT-Card"
 				(path "/cf02616b-7563-498d-8298-4a13535fe00b/26667293-4bc7-42dd-80bc-5789f6d81738"
 					(reference "R46")
@@
 		)
 		(instances
-			(project "myCC"
+			(project "CredIT-Card"
 				(path "/cf02616b-7563-498d-8298-4a13535fe00b/26667293-4bc7-42dd-80bc-5789f6d81738"
 					(reference "#PWR054")
@@
 		)
 		(instances
-			(project "myCC"
+			(project "CredIT-Card"
 				(path "/cf02616b-7563-498d-8298-4a13535fe00b/26667293-4bc7-42dd-80bc-5789f6d81738"
 					(reference "#PWR050")
@@
 		)
 		(instances
-			(project "myCC"
+			(project "CredIT-Card"
 				(path "/cf02616b-7563-498d-8298-4a13535fe00b/26667293-4bc7-42dd-80bc-5789f6d81738"
 					(reference "D1")
@@
 		)
 		(instances
-			(project "myCC"
+			(project "CredIT-Card"
 				(path "/cf02616b-7563-498d-8298-4a13535fe00b/26667293-4bc7-42dd-80bc-5789f6d81738"
 					(reference "#PWR058")
@@
 		)
 		(instances
-			(project "myCC"
+			(project "CredIT-Card"
 				(path "/cf02616b-7563-498d-8298-4a13535fe00b/26667293-4bc7-42dd-80bc-5789f6d81738"
 					(reference "#PWR053")
@@
 		)
 		(instances
-			(project "myCC"
+			(project "CredIT-Card"
 				(path "/cf02616b-7563-498d-8298-4a13535fe00b/26667293-4bc7-42dd-80bc-5789f6d81738"
 					(reference "R13")
@@
 		)
 		(instances
-			(project "myCC"
+			(project "CredIT-Card"
 				(path "/cf02616b-7563-498d-8298-4a13535fe00b/26667293-4bc7-42dd-80bc-5789f6d81738"
 					(reference "C19")
@@
 		)
 		(instances
-			(project "myCC"
+			(project "CredIT-Card"
 				(path "/cf02616b-7563-498d-8298-4a13535fe00b/26667293-4bc7-42dd-80bc-5789f6d81738"
 					(reference "#PWR056")
@@
 		)
 		(instances
-			(project "myCC"
+			(project "CredIT-Card"
 				(path "/cf02616b-7563-498d-8298-4a13535fe00b/26667293-4bc7-42dd-80bc-5789f6d81738"
 					(reference "C22")
@@
 		)
 		(instances
-			(project "myCC"
+			(project "CredIT-Card"
 				(path "/cf02616b-7563-498d-8298-4a13535fe00b/26667293-4bc7-42dd-80bc-5789f6d81738"
 					(reference "#PWR047")
@@
 		)
 		(instances
-			(project "myCC"
+			(project "CredIT-Card"
 				(path "/cf02616b-7563-498d-8298-4a13535fe00b/26667293-4bc7-42dd-80bc-5789f6d81738"
 					(reference "R14")
@@
 		)
 		(instances
-			(project "myCC"
+			(project "CredIT-Card"
 				(path "/cf02616b-7563-498d-8298-4a13535fe00b/26667293-4bc7-42dd-80bc-5789f6d81738"
 					(reference "TH1")
@@
 		)
 		(instances
-			(project "myCC"
+			(project "CredIT-Card"
 				(path "/cf02616b-7563-498d-8298-4a13535fe00b/26667293-4bc7-42dd-80bc-5789f6d81738"
 					(reference "#PWR062")
@@
 		)
 		(instances
-			(project "myCC"
+			(project "CredIT-Card"
 				(path "/cf02616b-7563-498d-8298-4a13535fe00b/26667293-4bc7-42dd-80bc-5789f6d81738"
 					(reference "#PWR042")
@@
 		)
 		(instances
-			(project "myCC"
+			(project "CredIT-Card"
 				(path "/cf02616b-7563-498d-8298-4a13535fe00b/26667293-4bc7-42dd-80bc-5789f6d81738"
 					(reference "R44")
@@
 		)
 		(instances
-			(project "myCC"
+			(project "CredIT-Card"
 				(path "/cf02616b-7563-498d-8298-4a13535fe00b/26667293-4bc7-42dd-80bc-5789f6d81738"
 					(reference "R15")
@@
 		)
 		(instances
-			(project "myCC"
+			(project "CredIT-Card"
 				(path "/cf02616b-7563-498d-8298-4a13535fe00b/26667293-4bc7-42dd-80bc-5789f6d81738"
 					(reference "C17")
@@
 		)
 		(instances
-			(project "myCC"
+			(project "CredIT-Card"
 				(path "/cf02616b-7563-498d-8298-4a13535fe00b/26667293-4bc7-42dd-80bc-5789f6d81738"
 					(reference "#PWR051")
@@
 		)
 		(instances
-			(project "myCC"
+			(project "CredIT-Card"
 				(path "/cf02616b-7563-498d-8298-4a13535fe00b/26667293-4bc7-42dd-80bc-5789f6d81738"
 					(reference "D2")
@@
 		)
 		(instances
-			(project "myCC"
+			(project "CredIT-Card"
 				(path "/cf02616b-7563-498d-8298-4a13535fe00b/26667293-4bc7-42dd-80bc-5789f6d81738"
 					(reference "#PWR059")
@@
 		)
 		(instances
-			(project "myCC"
+			(project "CredIT-Card"
 				(path "/cf02616b-7563-498d-8298-4a13535fe00b/26667293-4bc7-42dd-80bc-5789f6d81738"
 					(reference "R16")
@@
 	)
 	(symbol
-		(lib_id "myCC:XTPSM83100SIUR")
+		(lib_id "CredIT-Card:XTPSM83100SIUR")
 		(at 196.85 34.29 0)
 		(unit 1)
@@
 		)
 		(instances
-			(project "myCC"
+			(project "CredIT-Card"
 				(path "/cf02616b-7563-498d-8298-4a13535fe00b/26667293-4bc7-42dd-80bc-5789f6d81738"
 					(reference "U5")
@@
 		)
 		(instances
-			(project "myCC"
+			(project "CredIT-Card"
 				(path "/cf02616b-7563-498d-8298-4a13535fe00b/26667293-4bc7-42dd-80bc-5789f6d81738"
 					(reference "JP3")
@@
 		)
 		(instances
-			(project "myCC"
+			(project "CredIT-Card"
 				(path "/cf02616b-7563-498d-8298-4a13535fe00b/26667293-4bc7-42dd-80bc-5789f6d81738"
 					(reference "C18")
@@
 		)
 		(instances
-			(project "myCC"
+			(project "CredIT-Card"
 				(path "/cf02616b-7563-498d-8298-4a13535fe00b/26667293-4bc7-42dd-80bc-5789f6d81738"
 					(reference "#PWR064")
@@
 		)
 		(instances
-			(project "myCC"
+			(project "CredIT-Card"
 				(path "/cf02616b-7563-498d-8298-4a13535fe00b/26667293-4bc7-42dd-80bc-5789f6d81738"
 					(reference "C16")
@@
 		)
 		(instances
-			(project "myCC"
+			(project "CredIT-Card"
 				(path "/cf02616b-7563-498d-8298-4a13535fe00b/26667293-4bc7-42dd-80bc-5789f6d81738"
 					(reference "C21")
@@
 		)
 		(instances
-			(project "myCC"
+			(project "CredIT-Card"
 				(path "/cf02616b-7563-498d-8298-4a13535fe00b/26667293-4bc7-42dd-80bc-5789f6d81738"
 					(reference "R47")
@@
 		)
 		(instances
-			(project "myCC"
+			(project "CredIT-Card"
 				(path "/cf02616b-7563-498d-8298-4a13535fe00b/26667293-4bc7-42dd-80bc-5789f6d81738"
 					(reference "#PWR055")
@@
 		)
 		(instances
-			(project "myCC"
+			(project "CredIT-Card"
 				(path "/cf02616b-7563-498d-8298-4a13535fe00b/26667293-4bc7-42dd-80bc-5789f6d81738"
 					(reference "R45")
