File: PCB/SENSORS.kicad_sch (KiCad schematic)
At the start: 26 parts, among them U13 MPL3115A2S, U14 HDC3022-Q1, U15 OPT3004, U16 VL53L1CBV0FY-1, U17 ISM303DAC

Commit message: Renamed PCB project
Parts:
- U13: symbol myCC:MPL3115A2S -> CredIT-Card:MPL3115A2S
- U14: symbol myCC:HDC3022-Q1 -> CredIT-Card:HDC3022-Q1
- U15: symbol myCC:OPT3004 -> CredIT-Card:OPT3004
- U16: symbol myCC:VL53L1CBV0FY-1 -> CredIT-Card:VL53L1CBV0FY-1
- U17: symbol myCC:ISM303DAC -> CredIT-Card:ISM303DAC
