File: PCB/io.kicad_sch (KiCad schematic)
At the start: 66 parts, among them J1 SPEAKER, J2 LCD, J3 2295018-2, SW1 EG1215AA, SW2 2425578-1, SW3 2425578-1, U10 74LVC1G17, U11 MPR121QR2, U12 74LVC1G17, U6 AD5110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

Commit message: Renamed PCB project
Parts:
- D3: footprint myCC:GW DASPA2.EC -> CredIT-Card:GW DASPA2.EC
- J2: footprint myCC:TE_3-1734839-0 -> CredIT-Card:TE_3-1734839-0; symbol myCC:3-1734839-0 -> CredIT-Card:3-1734839-0
- J3: footprint myCC:TE_2295018-2 -> CredIT-Card:TE_2295018-2
- SW1: footprint myCC:SW_EG1215AA -> CredIT-Card:SW_EG1215AA
- SW2, SW3: footprint myCC:TE_2425578-1 -> CredIT-Card:TE_2425578-1
- TB1, TB2, TB3, TB4, TB5: footprint myCC:TOUCH_BT -> CredIT-Card:TOUCH_BT
- U6: symbol myCC:AD5110 -> CredIT-Card:AD5110
- U7: symbol myCC:LM27952SD -> CredIT-Card:LM27952SD
- U8: symbol myCC:LM4819 -> CredIT-Card:LM4819
- U9: symbol myCC:LTC3218 -> CredIT-Card:LTC3218
